Commit message: chore: Clean up application of forces and torques to use body

File: src/jdrones/envs/droneplus.urdf (robot description, URDF)
Before this commit: robot droneplus, 6 links, 5 joints
Links:
- removed link center_of_mass_link
Joints:
- removed joint center_of_mass_joint

Commit message: fix: Small changes to simplify drone model

File: src/jdrones/envs/droneplus.urdf (robot description, URDF)
Before this commit: robot droneplus, 5 links, 4 joints
Links:
- link base_link: mass None -> 1.4
